File: design/BLDC_4.sch (KiCad schematic (older format))
At the start: 26 parts, among them K1 SERVO, P1 HALL/Encoder, P101 CANBUS, P3 PWR_COMM, P4 IN+, P5 IN-, P6 MOTOR1, P7 MOTOR2, P9 MOTOR3, X1 MINI-USB-SHIELD-32005-201

Commit message: Initial commit of the DRV8312
Parts:
- removed C3: 100n, CRF1:SMD-0603_c, symbol C-RESCUE-BLDC_4
- removed K1: SERVO, CRF1:pinhead-1X03, symbol CONN_3
- removed P101: CANBUS, JST conn:b4b-ph-kl, symbol CONN_4
- removed R5: 2k2, CRF1:SMD-0603_r, symbol R-RESCUE-BLDC_4
Connections:
- wire segments 91 -> 78
Other:
- note removed: "100R if used as\nservo output"
- moved on the sheet: P9

Commit message: More updates to schematic.
Parts:
- removed C2: 100n, CRF1:SMD-0603_c, symbol C-RESCUE-BLDC_4
- removed R3: 39k, CRF1:SMD-0603_r, symbol R-RESCUE-BLDC_4
- removed R4: 2k2, CRF1:SMD-0603_r, symbol R-RESCUE-BLDC_4
- removed R53, R54: SHUNT, CRF1:WSLP2726, symbol SHUNT
Connections:
- wire segments 78 -> 53
Other:
- moved on the sheet: P6, P7, P9
