File: design/Power.sch (KiCad schematic (older format))
At the start: 48 parts, among them U2 TC2117, U3 DRV8302

Commit message: Initial commit of the DRV8312
Parts:
- removed C1, C39, C40, C43, C44, C49, C8, C9: 10u,50V, CRF1:SMD-1206, symbol C-RESCUE-BLDC_4
- removed C18, C20, C23, C24, C26, C52: 2.2u, CRF1:SMD-0603_c, symbol C-RESCUE-BLDC_4
- removed C19: 120p, CRF1:SMD-0603_c, symbol C-RESCUE-BLDC_4
- removed C21: 6.8n, CRF1:SMD-0603_c, symbol C-RESCUE-BLDC_4
- removed C22: 22n, CRF1:SMD-0603_c, symbol C-RESCUE-BLDC_4
- removed C25, C33: 100u, w_smd_cap:c_tant_B, symbol CP1-RESCUE-BLDC_4
- removed C27: 100n, CRF1:SMD-0603_c, symbol C-RESCUE-BLDC_4
- removed C28, C29, C30: 220n, CRF1:SMD-0603_c, symbol C-RESCUE-BLDC_4
- removed C34, C36: 2.2n, CRF1:SMD-0603_c, symbol C-RESCUE-BLDC_4
- removed C37: 15u,100V, w_smd_cap:c_2220, symbol C-RESCUE-BLDC_4
- removed C51: 15u, 100v, w_smd_cap:c_2220, symbol C-RESCUE-BLDC_4
- removed D4: DIODESCH, Diodes_SMD:SMA_Handsoldering, symbol DIODESCH
- removed D5: TVS 5V, w_smd_diode:do214ac, symbol DIODE
- removed R17: 18k, CRF1:SMD-0603_r, symbol R-RESCUE-BLDC_4
- removed R18: 3k3, CRF1:SMD-0603_r, symbol R-RESCUE-BLDC_4
- removed R19: 15k, CRF1:SMD-0603_r, symbol R-RESCUE-BLDC_4
- removed R20: 10k, CRF1:SMD-0603_r, symbol R-RESCUE-BLDC_4
- removed R21: 220k, CRF1:SMD-0603_r, symbol R-RESCUE-BLDC_4
- removed R23, R26, R32: 39k, CRF1:SMD-0603_r, symbol R-RESCUE-BLDC_4
- removed R24, R27, R33: 2k2, CRF1:SMD-0603_r, symbol R-RESCUE-BLDC_4
- removed R25: 1M, CRF1:SMD-0603_r, symbol R-RESCUE-BLDC_4
- removed R48, R49, R50, R51: 100R, CRF1:SMD-0603_r, symbol R-RESCUE-BLDC_4
- removed U2: TC2117, CRF1:SOT-223, symbol NCP1117ST33T3G
- removed U3: DRV8302, CRF1:TSSOP-56-PP, symbol DRV8302
- added C1, C18, C8: 1uF, symbol C
- added C19, C20, C3, C30, C33, C34, C44, C45, C46, C47, C9: 0.1uF, symbol C
- added C21, C22, C23, C36: 0.001uF, symbol C
- added C24, C25, C26, C27, C28, C29, C42, C43: 220pF, symbol C
- added C37, C39, C40: 0.047uF, symbol C
- added L2, L3: 4.7uH, symbol INDUCTOR
- added R14, R15, R16, R17, R18, R40, R41, R5: 1k, symbol R
- added R19, R20, R21: 28.7k, symbol R
- added R23, R24, R25, R43: 49.9k, symbol R
- added R26, R27, R28: 19.1k, symbol R
- added R29, R30, R31, R45: 33, symbol R
- added R32, R33, R34: 95.3k, symbol R
- added R35, R36, R39: 4.99k, symbol R
- added R42: 57.6k, symbol R
- added R44: 38.3k, symbol R
- added R46: 5m, symbol R
- added R47, R48, R49: 10m, symbol R
- added U2: DRV8312, NQBit:DRV8312, symbol DRV8312
- added U3, U4, U5, U6: OPA365AIDBV, TO_SOT_Packages_SMD:SOT-23-5, symbol OPA365AIDBV
- L1: value 22u -> 4.7uH; footprint w_smd_inductors:inductor_smd_8x5mm -> (none)
Connections:
- net labels added: +2V5, +3.3V, BST_A, BST_B, BST_C, GND_A, GND_B, GND_C, GND_TOTAL, GVDD, I_FDBK_A, I_FDBK_B, I_FDBK_C, I_FDBK_TOTAL, MOTOR_A, MOTOR_B, MOTOR_C, OUT_A, OUT_B, OUT_C, PVDD, V_FDBK_A, V_FDBK_B, V_FDBK_C
- net labels removed: +5V, BR_SO1, BR_SO2, DC_CAL, EN_GATE, FAULT, H1, H1_LOW, H1_VS, H2, H2_LOW, H2_VS, H3, H3_LOW, H3_VS, L1, L2, L3, M_H1, M_H2, M_H3, M_L1, M_L2, M_L3, SENS1, SENS2, SENS3, SH1_A, SH1_B, SH2_A, SH2_B, VCC, V_SUPPLY
- wire segments 189 -> 122
- no-connect marks 4 -> 0
Other:
- note added: "GVDD filter Caps for A, B, C"
- note added: "PVDD filter Caps for A, B, C"
- note removed: "3.3v regulator\nfor the logic"
- note removed: "MCU must sense the\nvoltage at each phase"

Commit message: More updates to schematic.
Parts:
- added C?: 0.1uF, symbol C
- added C?: 1uF, symbol C
- added C?: 47uF, symbol CP
- added C?: 100nF, symbol C
- added R?: 30k, symbol R
- added R?: 1, symbol R
- added R?: 39k, symbol R
- added R?: 2.2k, symbol R
Connections:
- net GND: now also U2.13 (GND), C?.2, C?.2, C?.2, R?.1, R?.1
- net GVDD: now also U2.2 (VDD), C?.1, C?.1
- net PVDD: now also R?.2
- net MODE_3: now reaches U2.10 (M3)
- net VREG: now reaches U2.11 (VREG)
- net VREG: now also C?.1
- net AGND: now reaches U2.12 (AGND)
- net AGND: now also C?.2, R?.1, R?.2
- net OC_ADJ: now reaches U2.14 (OC_ADJ)
- net OC_ADJ: now also R?.2
- net PWM_B: now reaches U2.15 (PWM_B)
- net RESET_A: now reaches U2.16 (RESET_A)
- net PWM_A: now reaches U2.17 (PWM_A)
- net FAULT: now reaches U2.18 (FAULT)
- net OTW: now reaches U2.21 (OTW)
- net PWM_C: now reaches U2.5 (PWM_C)
- net RESET_C: now reaches U2.6 (RESET_C)
- net RESET_B: now reaches U2.7 (RESET_B)
- net MODE_1: now reaches U2.8 (M1)
- net MODE_2: now reaches U2.9 (M2)
- new net V_FDBK_SUPPLY: C?.1, R?.1, R?.2
Other:
- note added: "Motor Driver Interface"
- moved on the sheet: R46, U2
